File: Optoisolated IR2184 & 6N137 daughter board.kicad_pcb (KiCad board)
At the start: 2 copper layers, 48.9 x 37.7 mm, 19 parts, among them J1 Screw_Terminal_01x08, U1 6N137, U2 IR2184, U3 LM78L05_TO92

Commit message: Update project files
Parts:
- removed H1, H2, H3, H4: MountingHole, MountingHole:MountingHole_3.2mm_M3
- moved R1 11.3 mm to (205.0, 52.5)
- moved J1 2.95 mm to (212.9, 78.4)
- moved C1 1.89 mm to (197.8, 55.7)
- moved R2 1.89 mm to (197.3, 58.9)
- moved U1 1.89 mm to (187.1, 52.9)
Routing:
- net /OPT_A: track 28.9 -> 10.8 mm
- net /OPT_K(GND): track 30.2 -> 36.2 mm
- net Net-(U1-A): track 7.60 -> 12.7 mm
- net /5V: track 45.7 -> 42.2 mm
- net /VO: track 37.1 -> 35.0 mm
- net /LO: track 31.0 -> 33.0 mm
- net GND: track 0.00 -> 1.98 mm, vias 11 -> 3
- net /VS: track 54.1 -> 55.8 mm
- net /12V_VCC: track 73.3 -> 74.7 mm
Other:
- board size 48.9 x 37.7 mm -> 41.3 x 31.6 mm

Commit message: Update project files
Parts:
- moved R4 14.0 mm to (206.1, 78.7), turned to 90 degrees
- moved R5 13.2 mm to (202.9, 78.7), turned to 90 degrees
- moved C3 11.5 mm to (190.1, 66.8), turned to 90 degrees
- moved C2 9.51 mm to (199.7, 71.4)
- moved U2 9.51 mm to (189.1, 71.5)
- moved R2 9.34 mm to (206.5, 60.5), turned to 90 degrees
- moved D1 7.96 mm to (186.7, 60.6), turned to 90 degrees
- moved R3 3.78 mm to (186.2, 70.9), turned to -90 degrees
- moved U1 2.43 mm to (189.4, 53.5)
- moved C1 2.18 mm to (200.0, 55.9), turned to 90 degrees
- moved R1 1.72 mm to (203.3, 53.0), turned to -90 degrees
Routing:
- net /VS: track 55.8 -> 26.8 mm, vias 2 -> 0
- net /LO: track 33.0 -> 8.07 mm
- net Net-(D1-K): track 34.0 -> 21.0 mm, vias 0 -> 4
- net /5V: track 42.2 -> 49.0 mm
- net /12V_VCC: track 74.7 -> 68.8 mm, vias 0 -> 7
- net /HO_R: track 13.0 -> 8.67 mm
- net /VO: track 35.0 -> 38.2 mm, vias 0 -> 2
- net Net-(U1-A): track 12.7 -> 15.8 mm
- net /OPT_A: track 10.8 -> 13.4 mm
- net /OPT_K(GND): track 36.2 -> 33.8 mm
- net Net-(U2-~{SD}): track 7.62 -> 5.74 mm
- net /HO: track 12.8 -> 11.3 mm
- net GND: vias 3 -> 1
Other:
- board size 41.3 x 31.6 mm -> 33.6 x 31.6 mm

Commit message: Update project files
Parts:
- removed C3: 0.1u, Capacitor_THT:C_Disc_D5.0mm_W2.5mm_P2.50mm
- moved R3 18.0 mm to (186.3, 52.9)
- moved D1 14.4 mm to (196.7, 70.9), turned to -90 degrees
- moved U2 2.53 mm to (186.6, 71.4)
Routing:
- net /12V_VCC: track 68.8 -> 53.2 mm, vias 7 -> 4
- net Net-(D1-K): track 21.0 -> 5.43 mm, vias 4 -> 0
- net /HO_R: track 8.67 -> 22.9 mm, vias 0 -> 1
- net Net-(U2-~{SD}): track 5.74 -> 14.7 mm
- net /VO: track 38.2 -> 30.4 mm
- net /5V: track 49.0 -> 53.6 mm, vias 0 -> 4
- net /VS: track 26.8 -> 24.7 mm
- net /LO_R: track 18.7 -> 20.7 mm

Commit message: Update project files
Routing:
- net /12V_VCC: track 53.2 -> 48.4 mm, vias 4 -> 2
- net /5V: track 53.6 -> 54.1 mm, vias 4 -> 2
Changed lines of the file:
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@@
   (segment (start 189.74 51.5) (end 191.69 53.45) (width 0.3) (layer "F.Cu") (net 1))
   (segment (start 202.97 58.9) (end 203.65 58.9) (width 0.3) (layer "F.Cu") (net 1))
+  (segment (start 205.91 62.96) (end 197.875 62.96) (width 0.3) (layer "F.Cu") (net 1))
+  (segment (start 197.875 62.96) (end 194.89 65.945) (width 0.3) (layer "F.Cu") (net 1))
   (segment (start 206.52 56.22) (end 206.52 52.9) (width 0.3) (layer "F.Cu") (net 1))
   (segment (start 203.88 58.9) (end 204.94 59.96) (width 0.3) (layer "F.Cu") (net 1))
   (segment (start 205.845 62.895) (end 207.06 64.11) (width 0.3) (layer "F.Cu") (net 1))
+  (segment (start 207.06 64.11) (end 205.91 62.96) (width 0.3) (layer "F.Cu") (net 1))
   (segment (start 197.14 55.92) (end 197.07 55.99) (width 0.3) (layer "F.Cu") (net 1))
   (segment (start 203.84 58.9) (end 206.52 56.22) (width 0.3) (layer "F.Cu") (net 1))
-  (segment (start 195.8 63.380001) (end 195.8 62.68) (width 0.3) (layer "F.Cu") (net 1))
-  (segment (start 194.89 64.290001) (end 195.8 63.380001) (width 0.3) (layer "F.Cu") (net 1))
   (segment (start 197.07 53.45) (end 197.07 55.99) (width 0.3) (layer "F.Cu") (net 1))
   (segment (start 186.35 52.29) (end 187.17 51.47) (width 0.3) (layer "F.Cu") (net 1))
@@
   (segment (start 191.69 53.45) (end 197.07 53.45) (width 0.3) (layer "F.Cu") (net 1))
   (segment (start 203.65 58.9) (end 203.88 58.9) (width 0.3) (layer "F.Cu") (net 1))
-  (segment (start 194.89 65.945) (end 194.89 64.290001) (width 0.3) (layer "F.Cu") (net 1))
-  (segment (start 201.86 62.49) (end 205.44 62.49) (width 0.3) (layer "F.Cu") (net 1))
   (segment (start 205.44 62.49) (end 207.06 64.11) (width 0.3) (layer "F.Cu") (net 1))
   (segment (start 204.94 59.96) (end 204.94 61.99) (width 0.3) (layer "F.Cu") (net 1))
@@
   (segment (start 186.35 52.89) (end 186.35 52.29) (width 0.3) (layer "F.Cu") (net 1))
   (segment (start 203.84 58.9) (end 203.65 58.9) (width 0.3) (layer "F.Cu") (net 1))
-  (via (at 201.86 62.49) (size 0.6) (drill 0.3) (layers "F.Cu" "B.Cu") (net 1))
-  (via (at 195.8 62.68) (size 0.6) (drill 0.3) (layers "F.Cu" "B.Cu") (net 1))
   (via (at 189.74 51.5) (size 0.6) (drill 0.3) (layers "F.Cu" "B.Cu") (net 1))
   (via (at 187.17 51.47) (size 0.6) (drill 0.3) (layers "F.Cu" "B.Cu") (net 1))
   (segment (start 189.71 51.47) (end 189.74 51.5) (width 0.3) (layer "B.Cu") (net 1))
-  (segment (start 201.67 62.68) (end 201.86 62.49) (width 0.3) (layer "B.Cu") (net 1))
-  (segment (start 195.8 62.68) (end 201.67 62.68) (width 0.3) (layer "B.Cu") (net 1))
   (segment (start 187.17 51.47) (end 189.71 51.47) (width 0.3) (layer "B.Cu") (net 1))
   (segment (start 212.97 74.92) (end 214.3 73.59) (width 0.3) (layer "F.Cu") (net 2))
@@
   (segment (start 203.135 65.945) (end 204.57 67.38) (width 0.3) (layer "F.Cu") (net 5))
   (segment (start 198.78 80.6) (end 199.67 80.6) (width 0.3) (layer "F.Cu") (net 5))
+  (segment (start 199.97 65.945) (end 197.535 68.38) (width 0.3) (layer "F.Cu") (net 5))
   (segment (start 199.97 65.945) (end 203.135 65.945) (width 0.3) (layer "F.Cu") (net 5))
   (segment (start 194.7 78.54) (end 194.21 79.03) (width 0.3) (layer "F.Cu") (net 5))
-  (segment (start 190.11 66.75) (end 193.53 63.33) (width 0.3) (layer "F.Cu") (net 5))
+  (segment (start 197.535 68.38) (end 192.95 68.38) (width 0.3) (layer "F.Cu") (net 5))
   (segment (start 196.72 78.54) (end 198.78 80.6) (width 0.3) (layer "F.Cu") (net 5))
-  (segment (start 196.48462 63.61462) (end 197.63962 63.61462) (width 0.3) (layer "F.Cu") (net 5))
-  (segment (start 197.63962 63.61462) (end 199.97 65.945) (width 0.3) (layer "F.Cu") (net 5))
+  (segment (start 190.11 75.34) (end 190.11 71.22) (width 0.3) (layer "F.Cu") (net 5))
+  (segment (start 192.95 68.38) (end 190.11 71.22) (width 0.3) (layer "F.Cu") (net 5))
   (segment (start 199.67 80.6) (end 210.69 80.6) (width 0.3) (layer "F.Cu") (net 5))
   (segment (start 192 77.23) (end 190.11 75.34) (width 0.3) (layer "F.Cu") (net 5))
-  (segment (start 193.53 63.33) (end 194.64 63.33) (width 0.3) (layer "F.Cu") (net 5))
-  (segment (start 190.11 75.34) (end 190.11 66.75) (width 0.3) (layer "F.Cu") (net 5))
   (via (at 192 77.23) (size 0.6) (drill 0.3) (layers "F.Cu" "B.Cu") (net 5))
   (via (at 192.24 78.84) (size 0.6) (drill 0.3) (layers "F.Cu" "B.Cu") (net 5))
-  (via (at 196.48462 63.61462) (size 0.6) (drill 0.3) (layers "F.Cu" "B.Cu") (net 5))
-  (via (at 194.64 63.33) (size 0.6) (drill 0.3) (layers "F.Cu" "B.Cu") (net 5))
-  (segment (start 196.2 63.33) (end 196.48462 63.61462) (width 0.3) (layer "B.Cu") (net 5))
   (segment (start 192.24 78.84) (end 192.24 77.47) (width 0.3) (layer "B.Cu") (net 5))
   (segment (start 192.24 77.47) (end 192 77.23) (width 0.3) (layer "B.Cu") (net 5))
-  (segment (start 194.64 63.33) (end 196.2 63.33) (width 0.3) (layer "B.Cu") (net 5))
   (segment (start 211.5 72.79) (end 212.87 71.42) (width 0.3) (layer "F.Cu") (net 6))
   (segment (start 204.65 72.79) (end 211.5 72.79) (width 0.3) (layer "F.Cu") (net 6))

Commit message: Update project files
Parts:
- removed C4: 0.1u, Capacitor_THT:C_Disc_D5.0mm_W2.5mm_P2.50mm
- moved R1 3.30 mm to (206.6, 53.0)
- moved R2 3.20 mm to (203.3, 60.6)
Routing:
- net /5V: track 54.1 -> 33.8 mm
- net /OPT_A: track 13.4 -> 8.09 mm
- net /VO: track 30.4 -> 26.0 mm, vias 2 -> 0
- net Net-(U1-A): track 15.8 -> 19.1 mm
