File: Optoisolated IR2184 & 6N137 daughter board.kicad_sch (KiCad schematic)
At the start: 16 parts, among them J1 Screw_Terminal_01x08, U1 6N137, U2 IR2184, U3 ADP7118ACPZN

Commit message: Update
Parts:
- C1: Manufacturer (none) -> Vishay; Manufacturer Part Number (none) -> VJ0805Y104JXAAT; Package (none) -> 0805; Supplier (none) -> Digikey; Supplier Part Number (none) -> 720-2029-1-ND; Voltage (none) -> 50v
- C2: footprint Capacitor_SMD:C_0805_2012Metric_Pad1.18x1.45mm_HandSolder -> Capacitor_SMD:C_1206_3216Metric_Pad1.33x1.80mm_HandSolder; Manufacturer (none) -> KYOCERA AVX; Manufacturer Part Number (none) -> 12065C105JAT2A; Package (none) -> 1206; Supplier (none) -> Digikey; Supplier Part Number (none) -> 478-KGM31HR71H105JUCT-ND; Voltage 25v -> 50v
- C3: value 0.1 -> 0.1u; Manufacturer (none) -> Vishay; Manufacturer Part Number (none) -> VJ0805Y104JXAAT; Package (none) -> 0805; Supplier (none) -> Digikey; Supplier Part Number (none) -> 720-2029-1-ND; Voltage (none) -> 50v
- C4: Manufacturer (none) -> Murata Electronics; Manufacturer Part Number (none) -> GRM21BR71C225KA12L; Package (none) -> 0805; Supplier (none) -> Digikey; Supplier Part Number (none) -> 490-3906-6-ND; Voltage (none) -> 16v
- C5, J1: Voltage (none) -> .
- C6: value 2.2 -> 2.2u; Manufacturer (none) -> Murata Electronics; Manufacturer Part Number (none) -> GRM21BR71C225KA12L; Package (none) -> 0805; Supplier (none) -> Digikey; Supplier Part Number (none) -> 490-3906-6-ND; Voltage (none) -> 16v
- D1: footprint Diode_SMD:D_0805_2012Metric_Pad1.15x1.40mm_HandSolder -> Diode_SMD:D_SOD-123; Manufacturer (none) -> Vishay; Manufacturer Part Number (none) -> 1N4148W-E3-08; Package (none) -> SOD-123; Supplier (none) -> Digikey; Supplier Part Number (none) -> 1N4148W-E3-08CT-ND; Voltage (none) -> .
- R1, R2: Manufacturer (none) -> TE connectivity; Manufacturer Part Number (none) -> CRG0805F470R; Package (none) -> 0805; Supplier (none) -> Digikey; Supplier Part Number (none) -> A106063CT-ND; Voltage (none) -> .
- R3: Manufacturer (none) -> TE Connectivity; Manufacturer Part Number (none) -> CRG0805F10K/10; Package (none) -> 0805; Supplier (none) -> Digikey; Supplier Part Number (none) -> A126332CT-ND; Voltage (none) -> .
- R4, R5: footprint Resistor_SMD:R_0805_2012Metric_Pad1.20x1.40mm_HandSolder -> Resistor_SMD:R_1206_3216Metric_Pad1.30x1.75mm_HandSolder; Manufacturer (none) -> TE connectivity; Manufacturer Part Number (none) -> CRGP1206F47R; Package (none) -> 1206; Supplier (none) -> Digikey; Supplier Part Number (none) -> A130522CT-ND; Voltage (none) -> .
- U1: Manufacturer (none) -> Vishay; Manufacturer Part Number (none) -> 6N137; Package (none) -> 8-DIP; Supplier (none) -> Digikey; Supplier Part Number (none) -> 751-1262-5-ND; Voltage (none) -> .
- U2: footprint Package_DIP:DIP-8_W7.62mm_LongPads -> Package_DIP:DIP-8_W8.89mm_SMDSocket_LongPads; Manufacturer (none) -> Infineon Technologies; Manufacturer Part Number (none) -> IR2184SPBF; Package (none) -> 8-SOIC; Supplier (none) -> Digikey; Supplier Part Number (none) -> IR2184SPBF-ND; Voltage (none) -> .
- U3: Manufacturer (none) -> Analoge device; Manufacturer Part Number (none) -> ADP7118ACPZN-R7; Package (none) -> 6-UDFN Exposed Pad; Supplier (none) -> Digikey; Supplier Part Number (none) -> 505-ADP7118ACPZN-R7CT-ND; Voltage (none) -> .

Commit message: PCB LAYOUT
Parts:
- removed C5: 1n, Capacitor_SMD:C_0805_2012Metric_Pad1.18x1.45mm_HandSolder, symbol Device:C
- removed U3: ADP7118ACPZN, Package_CSP:LFCSP-6-1EP_2x2mm_P0.65mm_EP1x1.6mm, symbol Regulator_Linear:ADP7118ACPZN
- added H1, H2, H3, H4: MountingHole, MountingHole:MountingHole_3.2mm_M3, symbol Mechanical:MountingHole
- added U3: LM78L05_TO92, Package_TO_SOT_THT:TO-220F-3_Vertical, symbol Regulator_Linear:LM78L05_TO92
- C1, C3: footprint Capacitor_SMD:C_0805_2012Metric_Pad1.18x1.45mm_HandSolder -> Capacitor_THT:C_Disc_D5.0mm_W2.5mm_P2.50mm; Manufacturer Vishay -> kemet; Manufacturer Part Number VJ0805Y104JXAAT -> C326C104K5R5TA; Package 0805 -> Radial; Supplier Part Number 720-2029-1-ND -> 399-9824-ND
- C2: footprint Capacitor_SMD:C_1206_3216Metric_Pad1.33x1.80mm_HandSolder -> Capacitor_THT:C_Disc_D5.0mm_W2.5mm_P2.50mm; Manufacturer KYOCERA AVX -> Murata Electronics; Manufacturer Part Number 12065C105JAT2A -> RDEC71E105K0P1H03B; Package 1206 -> Radial; Supplier Part Number 478-KGM31HR71H105JUCT-ND -> RDEC71E105K0P1H03B-ND; Voltage 50v -> 25v
- C4: value 2.2u -> 0.1u; footprint Capacitor_SMD:C_0805_2012Metric_Pad1.18x1.45mm_HandSolder -> Capacitor_THT:C_Disc_D5.0mm_W2.5mm_P2.50mm; Manufacturer Murata Electronics -> kemet; Manufacturer Part Number GRM21BR71C225KA12L -> C326C104K5R5TA; Package 0805 -> Radial; Supplier Part Number 490-3906-6-ND -> 399-9824-ND; Voltage 16v -> 50v
- C6: value 2.2u -> 0.22u; footprint Capacitor_SMD:C_0805_2012Metric_Pad1.18x1.45mm_HandSolder -> Capacitor_THT:C_Disc_D5.0mm_W2.5mm_P2.50mm; Manufacturer Murata Electronics -> Vishay; Manufacturer Part Number GRM21BR71C225KA12L -> K224Z15Y5VF5TL2; Package 0805 -> Radial; Supplier Part Number 490-3906-6-ND -> BC1161TR-ND; Voltage 16v -> 50v
- D1: footprint Diode_SMD:D_SOD-123 -> Diode_THT:D_DO-35_SOD27_P7.62mm_Horizontal; Manufacturer Part Number 1N4148W-E3-08 -> 1N4148-TAP; Package SOD-123 -> DO-35 Axial; Supplier Part Number 1N4148W-E3-08CT-ND -> 1N4148-TAPCT-ND
- R1, R2: footprint Resistor_SMD:R_0805_2012Metric_Pad1.20x1.40mm_HandSolder -> Resistor_THT:R_Axial_DIN0207_L6.3mm_D2.5mm_P7.62mm_Horizontal; Manufacturer Part Number CRG0805F470R -> CFR16J470R; Package 0805 -> Radial; Supplier Part Number A106063CT-ND -> A105933CT-ND
- R3: footprint Resistor_SMD:R_0805_2012Metric_Pad1.20x1.40mm_HandSolder -> Resistor_THT:R_Axial_DIN0207_L6.3mm_D2.5mm_P7.62mm_Horizontal; Manufacturer Part Number CRG0805F10K/10 -> CFR16J10K; Package 0805 -> Radial; Supplier Part Number A126332CT-ND -> A104668CT-ND
- R4, R5: footprint Resistor_SMD:R_1206_3216Metric_Pad1.30x1.75mm_HandSolder -> Resistor_THT:R_Axial_DIN0207_L6.3mm_D2.5mm_P7.62mm_Horizontal; Manufacturer Part Number CRGP1206F47R -> LR0204F47R; Package 1206 -> Radial; Supplier Part Number A130522CT-ND -> LR0204F47R-ND
- U2: footprint Package_DIP:DIP-8_W8.89mm_SMDSocket_LongPads -> Package_DIP:DIP-8_W7.62mm; Supplier Part Number IR2184SPBF-ND -> IR2184PBF-ND
Connections:
- net 12V_VCC: now also U3.3 (VI); no longer R3.1
- net 5V: now also R3.1, U3.1 (VO)
- net GND: now also U3.2 (GND)
Other:
- moved on the sheet: C1, C2, C3, C6, D1, J1, R1, R2, R3, R4, R5, U1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

Commit message: Update project files
Parts:
- removed H1, H2, H3, H4: MountingHole, MountingHole:MountingHole_3.2mm_M3, symbol Mechanical:MountingHole
Changed lines of the file:
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@@
     (effects (font (size 1.27 1.27)) (justify left bottom))
-  )
-  (symbol (lib_id "Mechanical:MountingHole") (at 114.3 83.82 0) (unit 1)
-    (in_bom yes) (on_board yes) (dnp no) (fields_autoplaced)
-    (property "Reference" "H2" (at 116.84 82.55 0)
-      (effects (font (size 1.27 1.27)) (justify left))
-    )
-    (property "Value" "MountingHole" (at 116.84 85.09 0)
-      (effects (font (size 1.27 1.27)) (justify left))
-    )
-    (property "Footprint" "MountingHole:MountingHole_3.2mm_M3" (at 114.3 83.82 0)
-      (effects (font (size 1.27 1.27)) hide)
-    )
-    (property "Datasheet" "~" (at 114.3 83.82 0)
-      (effects (font (size 1.27 1.27)) hide)
-    )
-    (instances
-      (project "Optoisolated IR2184 & 6N137 daughter board"
-        (path "/268f9dc7-5a94-4a9c-91d2-f40a19785bc2"
-          (reference "H2") (unit 1)
-        )
-      )
-    )
   )
   (symbol (lib_id "power:GND") (at 130.81 50.8 0) (unit 1)
@@
     )
   )
-  (symbol (lib_id "Mechanical:MountingHole") (at 114.3 95.25 0) (unit 1)
-    (in_bom yes) (on_board yes) (dnp no) (fields_autoplaced)
-    (property "Reference" "H4" (at 116.84 93.98 0)
-      (effects (font (size 1.27 1.27)) (justify left))
-    )
-    (property "Value" "MountingHole" (at 116.84 96.52 0)
-      (effects (font (size 1.27 1.27)) (justify left))
-    )
-    (property "Footprint" "MountingHole:MountingHole_3.2mm_M3" (at 114.3 95.25 0)
-      (effects (font (size 1.27 1.27)) hide)
-    )
-    (property "Datasheet" "~" (at 114.3 95.25 0)
-      (effects (font (size 1.27 1.27)) hide)
-    )
-    (instances
-      (project "Optoisolated IR2184 & 6N137 daughter board"
-        (path "/268f9dc7-5a94-4a9c-91d2-f40a19785bc2"
-          (reference "H4") (unit 1)
-        )
-      )
-    )
-  )
   (symbol (lib_id "Driver_FET:IR2184") (at 64.77 107.95 0) (unit 1)
     (in_bom yes) (on_board yes) (dnp no) (fields_autoplaced)
@@
         (path "/268f9dc7-5a94-4a9c-91d2-f40a19785bc2"
           (reference "C3") (unit 1)
-        )
-      )
-    )
-  )
-  (symbol (lib_id "Mechanical:MountingHole") (at 114.3 77.47 0) (unit 1)
-    (in_bom yes) (on_board yes) (dnp no) (fields_autoplaced)
-    (property "Reference" "H1" (at 116.84 76.2 0)
-      (effects (font (size 1.27 1.27)) (justify left))
-    )
-    (property "Value" "MountingHole" (at 116.84 78.74 0)
-      (effects (font (size 1.27 1.27)) (justify left))
-    )
-    (property "Footprint" "MountingHole:MountingHole_3.2mm_M3" (at 114.3 77.47 0)
-      (effects (font (size 1.27 1.27)) hide)
-    )
-    (property "Datasheet" "~" (at 114.3 77.47 0)
-      (effects (font (size 1.27 1.27)) hide)
-    )
-    (instances
-      (project "Optoisolated IR2184 & 6N137 daughter board"
-        (path "/268f9dc7-5a94-4a9c-91d2-f40a19785bc2"
-          (reference "H1") (unit 1)
         )
       )
@@
         )
       )
-    )
-  )
-  (symbol (lib_id "Mechanical:MountingHole") (at 114.3 88.9 0) (unit 1)
-    (in_bom yes) (on_board yes) (dnp no) (fields_autoplaced)
-    (property "Reference" "H3" (at 116.84 87.63 0)
-      (effects (font (size 1.27 1.27)) (justify left))
-    )
-    (property "Value" "MountingHole" (at 116.84 90.17 0)
-      (effects (font (size 1.27 1.27)) (justify left))
-    )
-    (property "Footprint" "MountingHole:MountingHole_3.2mm_M3" (at 114.3 88.9 0)
-      (effects (font (size 1.27 1.27)) hide)
-    )
-    (property "Datasheet" "~" (at 114.3 88.9 0)
-      (effects (font (size 1.27 1.27)) hide)
-    )
-    (instances
-      (project "Optoisolated IR2184 & 6N137 daughter board"
-        (path "/268f9dc7-5a94-4a9c-91d2-f40a19785bc2"
-          (reference "H3") (unit 1)
-        )
-      )

Commit message: Update project files
Parts:
- removed C3: 0.1u, Capacitor_THT:C_Disc_D5.0mm_W2.5mm_P2.50mm, symbol Device:C
Changed lines of the file:
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@@
   (junction (at 74.93 44.45) (diameter 0) (color 0 0 0 0)
-  )
-  (junction (at 55.88 91.44) (diameter 0) (color 0 0 0 0)
   )
   (no_connect (at 52.07 49.53))
@@
   )
   (wire (pts (xy 59.69 25.4) (xy 74.93 25.4))
-    (stroke (width 0) (type default))
-  )
-  (wire (pts (xy 50.8 91.44) (xy 55.88 91.44))
     (stroke (width 0) (type default))
   )
@@
     )
   )
-  (symbol (lib_id "power:GND") (at 50.8 99.06 0) (unit 1)
-    (in_bom yes) (on_board yes) (dnp no) (fields_autoplaced)
-    (property "Reference" "#PWR05" (at 50.8 105.41 0)
-      (effects (font (size 1.27 1.27)) hide)
-    )
-    (property "Value" "GND" (at 50.8 104.14 0)
-      (effects (font (size 1.27 1.27)))
-    )
-    (property "Footprint" "" (at 50.8 99.06 0)
-      (effects (font (size 1.27 1.27)) hide)
-    )
-    (property "Datasheet" "" (at 50.8 99.06 0)
-      (effects (font (size 1.27 1.27)) hide)
-    )
-    (pin "1")
-    (instances
-      (project "Optoisolated IR2184 & 6N137 daughter board"
-        (path "/268f9dc7-5a94-4a9c-91d2-f40a19785bc2"
-          (reference "#PWR05") (unit 1)
-        )
-      )
-    )
-  )
   (symbol (lib_id "Device:R") (at 33.02 41.91 90) (unit 1)
     (in_bom yes) (on_board yes) (dnp no) (fields_autoplaced)
@@
         )
       )
-    )
-  )
-  (symbol (lib_id "Device:C") (at 50.8 95.25 0) (mirror y) (unit 1)
-    (in_bom yes) (on_board yes) (dnp no)
-    (property "Reference" "C3" (at 46.99 93.98 0)
-      (effects (font (size 1.27 1.27)) (justify left))
-    )
-    (property "Value" "0.1u" (at 46.99 96.52 0)
-      (effects (font (size 1.27 1.27)) (justify left))
-    )
-    (property "Footprint" "Capacitor_THT:C_Disc_D5.0mm_W2.5mm_P2.50mm" (at 49.8348 99.06 0)
-      (effects (font (size 1.27 1.27)) hide)
-    )
-    (property "Datasheet" "https://content.kemet.com/datasheets/KEM_C1050_GOLDMAX_X7R.pdf" (at 50.8 95.25 0)
-      (effects (font (size 1.27 1.27)) hide)
-    )
-    (property "Manufacturer" "kemet" (at 50.8 95.25 0)
-      (effects (font (size 1.27 1.27)) hide)
-    )
-    (property "Manufacturer Part Number" "C326C104K5R5TA" (at 50.8 95.25 0)
-      (effects (font (size 1.27 1.27)) hide)
-    )
-    (property "Package" "Radial" (at 50.8 95.25 0)
-      (effects (font (size 1.27 1.27)) hide)
-    )
-    (property "Supplier" "Digikey" (at 50.8 95.25 0)
-      (effects (font (size 1.27 1.27)) hide)
-    )
-    (property "Supplier Part Number" "399-9824-ND" (at 50.8 95.25 0)
-      (effects (font (size 1.27 1.27)) hide)
-    )
-    (property "Voltage" "50v" (at 50.8 95.25 0)
-      (effects (font (size 1.27 1.27)) hide)
-    )
-    (pin "1")
-    (pin "2")
-    (instances
-      (project "Optoisolated IR2184 & 6N137 daughter board"
-        (path "/268f9dc7-5a94-4a9c-91d2-f40a19785bc2"
-          (reference "C3") (unit 1)
-        )
-      )

Commit message: Update project files
Parts:
- removed C4: 0.1u, Capacitor_THT:C_Disc_D5.0mm_W2.5mm_P2.50mm, symbol Device:C
Changed lines of the file:
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@@
-    (stroke (width 0) (type default))
-  )
-  (wire (pts (xy 138.43 31.75) (xy 143.51 31.75))
     (stroke (width 0) (type default))
   )
@@
   )
   (wire (pts (xy 20.32 41.91) (xy 29.21 41.91))
-    (stroke (width 0) (type default))
-  )
-  (wire (pts (xy 143.51 33.02) (xy 143.51 31.75))
     (stroke (width 0) (type default))
   )
@@
     (effects (font (size 1.27 1.27)) (justify left bottom))
   )
-  (label "5V" (at 143.51 31.75 0) (fields_autoplaced)
+  (label "5V" (at 138.43 31.75 0) (fields_autoplaced)
     (effects (font (size 1.27 1.27)) (justify left bottom))
   )
@@
         (path "/268f9dc7-5a94-4a9c-91d2-f40a19785bc2"
           (reference "R2") (unit 1)
-        )
-      )
-    )
-  )
-  (symbol (lib_id "power:GND") (at 143.51 40.64 0) (unit 1)
-    (in_bom yes) (on_board yes) (dnp no) (fields_autoplaced)
-    (property "Reference" "#PWR010" (at 143.51 46.99 0)
-      (effects (font (size 1.27 1.27)) hide)
-    )
-    (property "Value" "GND" (at 143.51 45.72 0)
-      (effects (font (size 1.27 1.27)))
-    )
-    (property "Footprint" "" (at 143.51 40.64 0)
-      (effects (font (size 1.27 1.27)) hide)
-    )
-    (property "Datasheet" "" (at 143.51 40.64 0)
-      (effects (font (size 1.27 1.27)) hide)
-    )
-    (pin "1")
-    (instances
-      (project "Optoisolated IR2184 & 6N137 daughter board"
-        (path "/268f9dc7-5a94-4a9c-91d2-f40a19785bc2"
-          (reference "#PWR010") (unit 1)
         )
       )
@@
         )
       )
-    )
-  )
-  (symbol (lib_id "Device:C") (at 143.51 36.83 0) (unit 1)
-    (in_bom yes) (on_board yes) (dnp no)
-    (property "Reference" "C4" (at 147.32 35.56 0)
-      (effects (font (size 1.27 1.27)) (justify left))
-    )
-    (property "Value" "0.1u" (at 147.32 38.1 0)
-      (effects (font (size 1.27 1.27)) (justify left))
-    )
-    (property "Footprint" "Capacitor_THT:C_Disc_D5.0mm_W2.5mm_P2.50mm" (at 144.4752 40.64 0)
-      (effects (font (size 1.27 1.27)) hide)
-    )
-    (property "Datasheet" "https://content.kemet.com/datasheets/KEM_C1050_GOLDMAX_X7R.pdf" (at 143.51 36.83 0)
-      (effects (font (size 1.27 1.27)) hide)
-    )
-    (property "Manufacturer" "kemet" (at 143.51 36.83 0)
-      (effects (font (size 1.27 1.27)) hide)
-    )
-    (property "Manufacturer Part Number" "C326C104K5R5TA" (at 143.51 36.83 0)
-      (effects (font (size 1.27 1.27)) hide)
-    )
-    (property "Package" "Radial" (at 143.51 36.83 0)
-      (effects (font (size 1.27 1.27)) hide)
-    )
-    (property "Supplier" "Digikey" (at 143.51 36.83 0)
-      (effects (font (size 1.27 1.27)) hide)
-    )
-    (property "Supplier Part Number" "399-9824-ND" (at 143.51 36.83 0)
-      (effects (font (size 1.27 1.27)) hide)
-    )
-    (property "Voltage" "50v" (at 143.51 36.83 0)
-      (effects (font (size 1.27 1.27)) hide)
-    )
-    (pin "2")
-    (pin "1")
-    (instances
-      (project "Optoisolated IR2184 & 6N137 daughter board"
-        (path "/268f9dc7-5a94-4a9c-91d2-f40a19785bc2"
-          (reference "C4") (unit 1)
-        )
-      )
